File: PCB/matrix.kicad_sch (KiCad schematic)
At the start: 169 parts

Commit message: PCB changes, readme, case files now added
- Changed MCU footprint from LQFP-48 to LQFP-48 + UFQFPN-48 dual footprint to combat MCU shortage
- PCB production files are for STM32F072CBUx; edit BOM, CPL, and paste layer if you want SMT assembly for an STM32F072CBTx
- STEP files and their associated technical drawings are now included for the case and plate
- Added more images, updated existing images
- Updated readme
Parts:
- D1, D10, D11, D12, D13, D14, D15, D16, D17, D18, D19, D2, D20, D21, D22, D23, D24, D25, D26, D27, D28, D29, D3, D30, D31, D32, D33, D34, D35, D36, D37, D38, D39, D4, D40, D41, D42, D43, D44, D45, D46, D47, D48, D49, D5, D50, D51, D52, D53, D54, D55, D56, D57, D58, D59, D6, D60, D61, D62, D63, D64, D65, D66, D67, D68, D69, D7, D70, D71, D72, D73, D74, D75, D8, D9: LCSC (none) -> C81598
- R4, R5: LCSC (none) -> C17557
